Commit message: tuning urdf to fit the real setting

File: urdf/realsense.urdf (robot description, URDF)
Before this commit: robot sawyer, 1 links, 1 joints
Joints:
- joint camera_link_base: origin xyz=0.025 0 0.25 rpy=0 0 0 -> xyz=0.015 0 0.275 rpy=0 0 0

Commit message: [bug fixed] * set status to 0 while detection failed * enlarge collision box in urdf

File: urdf/realsense.urdf (robot description, URDF)
Before this commit: robot sawyer, 1 links, 1 joints
Links:
- link camera_link: mass 0.0001 -> 0.072; geometry collision box size=0.32 0.32 0.32; visual mesh filename=package://openface_ros/meshes/d435.dae
